Commit message: Add ros2_control state interfaces for IMU
Signed-off-by: Ivan Santiago Paunovic <ivanpauno@ekumenlabs.com>

File: andino_description/urdf/include/andino_control.urdf.xacro (robot description, xacro)
@@ -29,4 +29,16 @@
       <state_interface name="position"/>
     </joint>
+    <sensor name="imu_sensor">
+      <state_interface name="imu_sensor/1"/>
+      <state_interface name="imu_sensor/2"/>
+      <state_interface name="imu_sensor/3"/>
+      <state_interface name="imu_sensor/4"/>
+      <state_interface name="imu_sensor/5"/>
+      <state_interface name="imu_sensor/6"/>
+      <state_interface name="imu_sensor/7"/>
+      <state_interface name="imu_sensor/8"/>
+      <state_interface name="imu_sensor/9"/>
+      <state_interface name="imu_sensor/10"/>
+    </joint>
   </ros2_control>
 </robot>

Commit message: Fix sensor tag closure in xacro file.

File: andino_description/urdf/include/andino_control.urdf.xacro (robot description, xacro)
@@ -40,5 +40,5 @@
       <state_interface name="imu_sensor/9"/>
       <state_interface name="imu_sensor/10"/>
-    </joint>
+    </sensor>
   </ros2_control>
 </robot>
